File: _autosave-qi-lamp-charger.sch (KiCad schematic (older format))
At the start: 7 parts

Commit message: Set up Qi schematic
Parts:
- U?: symbol qi-lamp-charger-rescue:BQ51050BYFP-Battery_Management -> Battery_Management:BQ51050BYFP
Changed lines of the file:
@@
 $EndComp
 $Comp
-L qi-lamp-charger-rescue:BQ51050BYFP-Battery_Management U?
+L Battery_Management:BQ51050BYFP U?
 U 1 1 6122ED8A
 P 5650 3450
