File: qi-lamp-charger.kicad_pcb (KiCad board)
At the start: 2 copper layers, 44 x 44 mm, 85 parts, among them J1 Conn_01x02, J2 Conn_01x02, J3 Conn_01x02, J4 Conn_01x06, J5 Conn_01x03, Q1 BSS308PE H6327, SW1 SKTDLDE010, U1 SLG5NV1430V, U2 BQ51050BYFP, U3 ESP-12E

Commit message: Layout proposal 2
Parts:
- C24, C25, C26, C27, C28, C29, C30, C31, C32, C33, JP10, JP11, JP12, JP13, JP14, JP5, JP6, JP7, JP8, JP9: moved to F.Cu
- moved JP9 80.2 mm to (85.3, 108.5), turned to 120 degrees
- moved JP8 79.6 mm to (100.0, 117.0)
- moved JP14 79.4 mm to (92.0, 100.0), turned to 90 degrees
- moved JP13 77.4 mm to (100.0, 108.0)
- moved C27 75.6 mm to (95.6, 114.6), turned to 90 degrees
- moved JP10 73.0 mm to (85.3, 91.5), turned to 60 degrees
- moved C32 69.7 mm to (95.6, 105.6), turned to 90 degrees
- moved JP12 68.3 mm to (108.0, 100.0), turned to -90 degrees
- moved C28 68.1 mm to (90.7, 109.3), turned to 0 degrees
- moved C30 66.2 mm to (104.4, 94.4), turned to -90 degrees
- moved JP7 64.4 mm to (114.7, 108.5), turned to -120 degrees
- moved JP11 60.9 mm to (100.0, 92.0), turned to 0 degrees
- moved C31 59.6 mm to (105.6, 104.4)
- moved C26 59.3 mm to (110.1, 110.8), turned to 150 degrees
- moved JP5 58.8 mm to (100.0, 83.0), turned to 0 degrees
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Routing:
- net /LED_VCC: track 0.00 -> 112.8 mm
- net Net-(D5-Pad4): track 15.9 -> 34.8 mm, vias 0 -> 2
- net Net-(D7-Pad4): track 10.2 -> 13.7 mm
- net Net-(D9-Pad4): track 10.2 -> 13.7 mm
- net Net-(D9-Pad2): track 10.2 -> 13.7 mm
- net Net-(D6-Pad4): track 16.2 -> 19.5 mm
- net Net-(D2-Pad4): track 15.9 -> 19.1 mm
- net Net-(D4-Pad4): track 15.4 -> 18.4 mm
- net Net-(D3-Pad4): track 16.2 -> 19.1 mm
- net /LED_DOUT: track 0.00 -> 2.46 mm
- net /LED_DIN: track 0.00 -> 2.46 mm
- net Net-(D1-Pad4): track 17.8 -> 18.4 mm
- added copper zone on B.Cu, net GND
- added copper zone on F.Cu, net GND

Commit message: Layout Qi
Parts:
- removed JP15, JP2: SolderJumper_2_Open, Jumper:SolderJumper-2_P1.3mm_Open_RoundedPad1.0x1.5mm
- removed JP3: SolderJumper_2_Bridged, Jumper:SolderJumper-2_P1.3mm_Bridged_RoundedPad1.0x1.5mm
- added TP1: TestPoint_2Pole, Connector_PinHeader_2.54mm:PinHeader_1x02_P2.54mm_Vertical, F.Cu at (172.4, 67.1)
- R14: value 100k -> 1M
- U2: value BQ51050BYFP -> BQ51050BRHL; footprint Package_BGA:Texas_DSBGA-28_1.9x3.0mm_Layout4x7_P0.4mm -> Package_DFN_QFN:Texas_VQFN-RHL-20
- moved C23 83.4 mm to (158.0, 136.0), turned to -90 degrees
- moved J5 70.7 mm to (156.0, 133.0)
- moved D11 68.1 mm to (167.0, 113.0), turned to 90 degrees
- moved R5 67.6 mm to (150.9, 115.5)
- moved R4 67.4 mm to (167.0, 116.0), turned to 90 degrees
- moved C20 63.5 mm to (138.0, 111.0), turned to -90 degrees
- moved C6 61.2 mm to (153.0, 105.0), turned to -90 degrees
- moved C21 60.5 mm to (136.0, 111.0), turned to -90 degrees
- moved C17 56.7 mm to (146.1, 109.2), turned to -90 degrees
- moved Q1 56.6 mm to (184.0, 89.0), turned to -90 degrees
- moved C13 56.6 mm to (144.5, 117.5), turned to -90 degrees
- moved C5 56.2 mm to (163.5, 124.0), turned to -90 degrees
- moved J3 56.0 mm to (140.5, 120.5), turned to -90 degrees
- moved D12 55.6 mm to (182.0, 93.0)
- moved C2 55.5 mm to (150.0, 104.0)
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Connections:
- net /DTR renamed DTR
- net /ESP_GPIO0 renamed ESP_GPIO0
- net /ESP_ON/~{OFF} renamed PWR_ON/~{OFF}
- net /ESP_RXD renamed ESP_RXD
- net /ESP_TXD renamed ESP_TXD
- net /LED_DIN renamed LED_DIN
- net /LED_DOUT renamed LED_DOUT
- net /Qi_NTC renamed Qi_NTC
- net /RTS renamed RTS
- net /~{ESP_RST} renamed ~{ESP_RST}
- C13 pad 1: Net-(U2-PadF1) -> Net-(C13-Pad1)
- C22 pad 1: VCC -> +VSW
- C23 pad 1: VCC -> LED_V+
- C24 pad 1: /LED_VCC -> LED_V+
- C25 pad 1: /LED_VCC -> GND
- C25 pad 2: GND -> LED_V+
- C26 pad 1: /LED_VCC -> LED_V+
- C27 pad 1: /LED_VCC -> LED_V+
- C28 pad 1: /LED_VCC -> LED_V+
- C29 pad 1: /LED_VCC -> LED_V+
- C30 pad 1: /LED_VCC -> GND
- C30 pad 2: GND -> LED_V+
- C31 pad 1: /LED_VCC -> GND
- C31 pad 2: GND -> LED_V+
- C32 pad 1: /LED_VCC -> GND
- C32 pad 2: GND -> LED_V+
- C33 pad 1: /LED_VCC -> GND
- C33 pad 2: GND -> LED_V+
- C34 pad 1: VCC -> +VSW
- D1 pad 3: /LED_VCC -> LED_V+
- D10 pad 3: /LED_VCC -> LED_V+
- D11 pad 2: +BATT -> +VSW
- D2 pad 3: /LED_VCC -> LED_V+
- D3 pad 3: /LED_VCC -> LED_V+
- D4 pad 3: /LED_VCC -> LED_V+
- D5 pad 3: /LED_VCC -> LED_V+
- D6 pad 3: /LED_VCC -> LED_V+
- D7 pad 3: /LED_VCC -> LED_V+
- D8 pad 3: /LED_VCC -> LED_V+
- D9 pad 3: /LED_VCC -> LED_V+
- J2 pad 1: Net-(C1-Pad1) -> Net-(C14-Pad2)
- J2 pad 2: Net-(C14-Pad2) -> Net-(C1-Pad1)
- J4 pad 3: /3V3 -> unconnected-(J4-Pad3)
- J5 pad 1: VCC -> LED_V+
- JP4 pad 1: VCC -> +VSW
- JP4 pad 2: /LED_VCC -> LED_V+
- R10 pad 2: VCC -> +VSW
- R11 pad 2: VCC -> +VSW
- R2 pad 2: Net-(U2-PadF1) -> Net-(C13-Pad1)
- R3 pad 1: Net-(U2-PadF1) -> Net-(C13-Pad1)
- R4 pad 1: /~{Qi_CHG} -> ~{Qi_CHG/LED}
- R6 pad 1: Net-(U2-PadF1) -> Net-(C13-Pad1)
- R9 pad 2: VCC -> +VSW
- U1 pad 1: Net-(U1-Pad1) -> +BATT
- U1 pad 5: VCC -> +VSW
- U1 pad 6: VCC -> +VSW
- U3 pad 20: /~{Qi_CHG} -> ~{Qi_CHG/LED}
- U3 pad 8: VCC -> +VSW
Routing:
- net LED_V+: track 0.00 -> 118.3 mm
- net /LED_VCC: track 112.8 -> 0.00 mm
- net Net-(D5-Pad4): track 34.8 -> 19.1 mm, vias 2 -> 0
- net GND: track 0.00 -> 15.4 mm, vias 0 -> 2
- net Net-(C1-Pad2): track 0.00 -> 14.8 mm
- net Net-(D2-Pad4): track 19.1 -> 33.1 mm, vias 0 -> 2
- net Net-(C14-Pad2): track 0.00 -> 13.5 mm
- net Net-(C1-Pad1): track 0.00 -> 11.6 mm
- net Net-(C10-Pad1): track 0.00 -> 5.86 mm
- net Net-(C18-Pad2): track 0.00 -> 5.78 mm
- net Net-(C9-Pad1): track 0.00 -> 4.15 mm
- net Net-(C19-Pad2): track 0.00 -> 4.07 mm
- net +BATT: track 0.00 -> 3.40 mm, vias 0 -> 1
- net Net-(C17-Pad2): track 0.00 -> 2.40 mm
- net +VSW: track 0.00 -> 1.91 mm
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
Commit message: Modules built
Parts:
- R3: value R -> 464k
- R6: value R -> 10k
- moved JP4 94.9 mm to (85.5, 66.4)
- moved C22 86.6 mm to (97.9, 128.1)
- moved R13 81.5 mm to (102.4, 132.9)
- moved R9 78.7 mm to (96.4, 132.4)
- moved C34 78.6 mm to (102.7, 128.9)
- moved R11 33.6 mm to (159.4, 69.2)
- moved JP1 33.2 mm to (160.8, 74.5)
- moved D12 30.7 mm to (159.7, 71.9)
- moved R8 28.5 mm to (143.9, 113.5)
- moved R10 19.8 mm to (159.9, 67.2)
- moved J3 7.38 mm to (147.0, 124.0), turned to 0 degrees
- moved R6 6.81 mm to (142.8, 124.3)
- moved C13 6.80 mm to (144.4, 124.3)
- moved R2 6.75 mm to (143.6, 120.4), turned to 180 degrees
- moved R3 5.46 mm to (143.6, 122.0), turned to 0 degrees
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Connections:
- C13 pad 1: Net-(C13-Pad1) -> Qi_TS/CTRL
- J3 pad 1: Qi_NTC -> GND
- J3 pad 2: GND -> Qi_NTC
- R2 pad 2: Net-(C13-Pad1) -> Qi_TS/CTRL
- R3 pad 1: Net-(C13-Pad1) -> Qi_TS/CTRL
- R6 pad 1: Net-(C13-Pad1) -> Qi_TS/CTRL
- U2 pad 11: GND -> unconnected-(U2-Pad11)
- U2 pad 13: Net-(C13-Pad1) -> Qi_TS/CTRL
- U3 pad 7: unconnected-(U3-Pad7) -> Qi_TS/CTRL
Routing:
- net GND: track 15.4 -> 17.1 mm
- net Qi_TS/CTRL: track 0.00 -> 1.58 mm
- net Net-(C13-Pad1): track 1.58 -> 0.00 mm
- net +BATT: track 3.40 -> 4.94 mm
- net Net-(R1-Pad2): track 1.44 -> 2.83 mm
- net PWR_ON/~{OFF}: track 0.00 -> 1.36 mm
- net Net-(C12-Pad1): track 0.00 -> 1.36 mm

Commit message: Moving in
Parts:
- C20, C21, C3: moved to F.Cu
- moved C12 121.0 mm to (79.0, 114.0), turned to 0 degrees
- moved U1 120.8 mm to (78.0, 116.0), turned to 180 degrees
- moved C16 118.1 mm to (79.0, 118.0), turned to 0 degrees
- moved SW1 103.2 mm to (81.8, 100.0), turned to 90 degrees
- moved R14 101.7 mm to (83.3, 95.5), turned to 90 degrees
- moved C23 91.7 mm to (100.3, 64.8), turned to 180 degrees
- moved J5 84.5 mm to (102.8, 67.4), turned to 90 degrees
- moved C10 64.5 mm to (92.0, 116.3), turned to -90 degrees
- moved C9 61.6 mm to (93.5, 116.3), turned to -90 degrees
- moved C11 58.6 mm to (95.0, 116.3), turned to -90 degrees
- moved R5 56.4 mm to (94.7, 110.7)
- moved C15 52.3 mm to (98.9, 118.1), turned to 90 degrees
- moved U2 52.1 mm to (98.0, 113.3), turned to 0 degrees
- moved C14 51.2 mm to (100.4, 118.1), turned to 90 degrees
- moved C6 50.9 mm to (103.8, 117.9), turned to -75 degrees
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- renumbered JP5 to JP1, JP14 to JP10, JP4 to JP11, JP1 to JP12, JP6 to JP2, JP7 to JP3, JP8 to JP4, JP9 to JP5, JP10 to JP6, JP11 to JP7, JP12 to JP8, JP13 to JP9
Routing:
- net LED_V+: track 118.3 -> 61.0 mm
- net LED_DOUT: track 2.46 -> 24.6 mm, vias 0 -> 1
- net GND: track 17.1 -> 35.3 mm, vias 2 -> 5
- net Net-(D3-Pad4): track 19.1 -> 5.02 mm
- net Net-(D5-Pad4): track 19.1 -> 5.16 mm
- net Net-(D4-Pad4): track 18.4 -> 5.06 mm
- net Net-(C20-Pad1): track 1.25 -> 10.6 mm, vias 1 -> 2
- net Qi_TS/CTRL: track 1.58 -> 10.4 mm
- net LED_DIN: track 2.46 -> 11.1 mm, vias 0 -> 1
- net Net-(C14-Pad2): track 13.5 -> 18.6 mm
- net Net-(C1-Pad1): track 11.6 -> 6.97 mm
- net Net-(R5-Pad1): track 0.00 -> 2.15 mm
- net ~{Qi_CHG/LED}: track 0.00 -> 1.85 mm
- net Net-(R1-Pad2): track 2.83 -> 4.64 mm
Other:
- board size 44 x 44 mm -> 41.5 x 44 mm

Commit message: Puzzling
Parts:
- removed J3: Conn_01x02, Connector_PinHeader_2.54mm:PinHeader_1x02_P2.54mm_Vertical
- J1: value Conn_01x02 -> Conn_01x03; footprint Connector_PinHeader_2.54mm:PinHeader_1x02_P2.54mm_Vertical -> Connector_PinHeader_2.54mm:PinHeader_1x03_P2.54mm_Vertical
- moved J4 89.1 mm to (85.9, 99.2), turned to -30 degrees
- moved J1 76.0 mm to (90.4, 115.9), turned to 52.5 degrees
- moved D12 74.4 mm to (89.8, 97.4), turned to 0 degrees
- moved R11 61.4 mm to (101.5, 89.5), turned to 90 degrees
- moved TP1 45.0 mm to (127.5, 70.0), turned to 180 degrees
- moved JP12 31.3 mm to (130.0, 68.7), turned to -90 degrees
- moved R10 27.6 mm to (132.3, 68.7), turned to 90 degrees
- moved C13 24.6 mm to (139.9, 138.0)
- moved C4 24.6 mm to (137.5, 121.5)
- moved C5 24.6 mm to (139.0, 121.5)
- moved C8 24.6 mm to (160.5, 83.5)
- moved D11 24.6 mm to (142.5, 110.5)
- moved Q1 24.6 mm to (159.5, 86.5)
- moved R12 24.6 mm to (161.5, 87.5)
- moved R2 24.6 mm to (139.1, 134.1)
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Connections:
- C27 pad 1: LED_V+ -> GND
- C27 pad 2: GND -> LED_V+
- J1 pad 2: GND -> NTC
- R3 pad 2: Qi_NTC -> NTC
- U3 pad 11: unconnected-(U3-Pad11) -> ~{Qi_CHG/LED}
- U3 pad 2: Qi_NTC -> NTC
- U3 pad 20: ~{Qi_CHG/LED} -> unconnected-(U3-Pad20)
Routing:
- net NTC: track 0.00 -> 47.7 mm
- net LED_V+: track 61.0 -> 34.4 mm, vias 0 -> 1
- net ESP_TXD: track 0.00 -> 23.7 mm
- net ESP_RXD: track 0.00 -> 23.4 mm
- net GND: track 35.3 -> 16.0 mm, vias 5 -> 7
- net Net-(D6-Pad4): track 19.5 -> 5.02 mm
- net ~{Qi_CHG/LED}: track 1.85 -> 15.3 mm, vias 0 -> 2
- net +BATT: track 4.94 -> 18.3 mm, vias 1 -> 2
- net DTR: track 0.00 -> 4.63 mm
- net +VSW: track 1.48 -> 5.42 mm
- net Net-(C1-Pad2): track 14.8 -> 18.5 mm
- net LED_DOUT: track 24.6 -> 22.8 mm
- net Net-(C11-Pad1): track 1.75 -> 2.76 mm
- net Net-(C20-Pad1): track 10.6 -> 9.74 mm
- net Net-(R5-Pad1): track 2.15 -> 1.34 mm

Commit message: Puzzling #2
Parts:
- TP1: footprint Connector_PinHeader_2.54mm:PinHeader_1x02_P2.54mm_Vertical -> Connector_PinHeader_1.00mm:PinHeader_1x02_P1.00mm_Vertical; moved to B.Cu
- moved R10 45.1 mm to (88.3, 78.5)
- moved JP12 44.9 mm to (86.2, 78.5)
- moved TP1 44.7 mm to (83.7, 79.0), turned to 0 degrees
- moved J1 4.66 mm to (86.6, 113.2), turned to -127.5 degrees
- moved C32 3.22 mm to (97.5, 104.6), turned to 0 degrees
- moved C28 2.47 mm to (83.9, 104.2), turned to -150 degrees
- moved R14 1.13 mm to (88.2, 100.5), turned to -120 degrees
- moved R11 0.81 mm to (102.3, 89.6), turned to 0 degrees
- moved D12 0.30 mm to (89.8, 97.7), turned to 60 degrees
Connections:
- J1 pad 1: +BATT -> GND
- J1 pad 3: GND -> +BATT
Routing:
- net +VSW: track 5.42 -> 32.3 mm, vias 0 -> 2
- net PWR_ON/~{OFF}: track 1.57 -> 27.1 mm
- net ESP_GPIO0: track 0.00 -> 19.4 mm
- net GND: track 16.0 -> 29.1 mm, vias 7 -> 23
- net NTC: track 47.7 -> 40.7 mm
- net DTR: track 4.63 -> 9.05 mm
- net Net-(D1-Pad4): track 18.4 -> 19.8 mm
- net Net-(D8-Pad4): track 15.1 -> 13.7 mm, vias 0 -> 2
- net ESP_RXD: track 23.4 -> 22.1 mm
- net ESP_TXD: track 23.7 -> 22.4 mm
Other:
- board text added: "Qi WiFi Lamp Step7.dk"

Commit message: Puzzling #3
Parts:
- TP1: footprint Connector_PinHeader_1.00mm:PinHeader_1x02_P1.00mm_Vertical -> Connector_PinHeader_1.27mm:PinHeader_1x02_P1.27mm_Vertical
- moved C8 89.2 mm to (72.7, 99.3)
- moved Q1 89.2 mm to (71.7, 102.3)
- moved R12 89.2 mm to (73.7, 103.3)
- moved R2 59.4 mm to (89.6, 101.3), turned to 60 degrees
- moved C4 47.9 mm to (90.3, 113.6), turned to 142.5 degrees
- moved C5 47.0 mm to (92.7, 113.7), turned to 45 degrees
- moved R13 43.2 mm to (97.3, 90.0), turned to 0 degrees
- moved JP11 42.9 mm to (83.9, 109.3), turned to 120 degrees
- moved C13 40.8 mm to (107.2, 113.6), turned to 180 degrees
- moved R6 40.5 mm to (107.2, 112.1), turned to 180 degrees
- moved R3 37.2 mm to (110.3, 112.1)
- moved R9 25.4 mm to (108.7, 110.2)
- moved C34 24.7 mm to (92.1, 106.6), turned to 90 degrees
- moved C22 23.0 mm to (90.3, 106.4), turned to 90 degrees
- moved C23 19.5 mm to (103.3, 84.0), turned to -90 degrees
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Connections:
- C26 pad 1: LED_V+ -> GND
- C26 pad 2: GND -> LED_V+
- C30 pad 1: GND -> LED_V+
- C30 pad 2: LED_V+ -> GND
Routing:
- net LED_V+: track 34.6 -> 100.6 mm, vias 1 -> 4
- net Qi_TS/CTRL: track 10.4 -> 47.0 mm, vias 0 -> 2
- net +VSW: track 32.3 -> 62.3 mm
- net +BATT: track 18.6 -> 34.8 mm, vias 2 -> 3
- net Net-(D1-Pad4): track 19.8 -> 5.06 mm
- net LED_DIN: track 11.1 -> 21.3 mm, vias 1 -> 2
- net RTS: track 0.00 -> 9.23 mm
- net GND: track 29.1 -> 38.0 mm, vias 23 -> 27
- net Net-(R9-Pad1): track 0.00 -> 6.73 mm
- net PWR_ON/~{OFF}: track 27.1 -> 29.9 mm, vias 0 -> 2
- net Net-(R13-Pad2): track 0.00 -> 2.66 mm
- net ~{ESP_RST}: track 0.00 -> 1.65 mm
- net Net-(D8-Pad4): track 13.7 -> 15.0 mm
- net Net-(C14-Pad2): track 18.6 -> 17.7 mm
- net Net-(C1-Pad1): track 6.97 -> 6.07 mm
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
Commit message: Puzzling #4
Parts:
- moved C8 15.8 mm to (87.2, 105.5), turned to 90 degrees
- moved Q1 13.4 mm to (84.7, 105.5)
- moved R12 8.78 mm to (82.2, 105.5)
Routing:
- net Net-(D5-Pad4): track 5.16 -> 19.6 mm
- net PWR_ON/~{OFF}: track 29.9 -> 42.0 mm, vias 2 -> 3
- net DTR: track 9.05 -> 17.0 mm
- net Net-(Q1-Pad3): track 0.00 -> 2.55 mm
- net LED_V+: track 100.6 -> 101.3 mm
- net GND: vias 27 -> 28
