File: qi-lamp-charger.kicad_sch (KiCad schematic)
At the start: 83 parts, among them J1 Conn_01x02, J2 Conn_01x02, J3 Conn_01x02, J4 Conn_01x06, J5 Conn_01x03, Q1 BSS308PE H6327, SW1 SKTDLDE010, U1 SLG5NV1430V, U2 BQ51050BRHL, U3 ESP-12E

Commit message: Modules built
Parts:
- C13: Name C_{3} -> C_{3NTC}
- R2: Name (none) -> R_{2NTC}; fit_field (none) -> DNP
- R3: value R -> 464k; Name (none) -> R_{1NTC}; fit_field (none) -> DNP
- R6: value R -> 10k; Name (none) -> R_{3NTC}
Connections:
- net GND: now also J3.1 (Pin_1); no longer J3.2 (Pin_2), U2.11 (EN2)
- net Qi_NTC: now also J3.2 (Pin_2); no longer J3.1 (Pin_1)
- net Qi_TS/CTRL: now reaches U3.7 (GPIO13)
- net Qi_TS/CTRL: now also C13.1, R2.2, R3.1, R6.1, U2.13 (TS/CTRL)
Other:
- note added: "Design for NTC: NTC β = 3534 NTC Ro = 10 kΩ R_{1} = 200 Ω R_{2} = 20 kΩ R_{3} = 464 kΩ No NTC: R_{2} = DNP R_{3} = 10 kΩ"
Changed lines of the file:
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@@
   (junction (at 57.15 142.24) (diameter 0) (color 0 0 0 0)
   )
+  (no_connect (at 147.32 60.96))
   (no_connect (at 121.92 38.1))
   (no_connect (at 359.41 138.43))
@@
   (no_connect (at 177.8 156.21))
   (no_connect (at 177.8 151.13))
-  (no_connect (at 177.8 148.59))
   (wire (pts (xy 278.13 116.84) (xy 269.24 116.84))
     (stroke (width 0) (type default) (color 0 0 0 0))
@@
     (stroke (width 0) (type default) (color 0 0 0 0))
   )
+  (wire (pts (xy 177.8 148.59) (xy 193.04 148.59))
+    (stroke (width 0) (type default) (color 0 0 0 0))
+  )
   (wire (pts (xy 172.72 66.04) (xy 172.72 68.58))
     (stroke (width 0) (type default) (color 0 0 0 0))
@@
     (stroke (width 0) (type default) (color 0 0 0 0))
   )
+  (wire (pts (xy 220.98 64.77) (xy 231.14 64.77))
+    (stroke (width 0) (type default) (color 0 0 0 0))
+  )
   (wire (pts (xy 90.17 48.26) (xy 90.17 49.53))
     (stroke (width 0) (type default) (color 0 0 0 0))
@@
     (stroke (width 0) (type default) (color 0 0 0 0))
   )
-  (wire (pts (xy 147.32 60.96) (xy 177.8 60.96))
-    (stroke (width 0) (type default) (color 0 0 0 0))
-  )
   (wire (pts (xy 212.09 64.77) (xy 220.98 64.77))
     (stroke (width 0) (type default) (color 0 0 0 0))
@@
     (effects (font (size 1.27 1.27)) (justify left bottom))
   )
+  (text "Design for NTC:\nNTC β = 3534\nNTC Ro = 10 kΩ\nR_{1} = 200 Ω\nR_{2} =  20 kΩ\nR_{3} = 464 kΩ\n\nNo NTC:\nR_{2} = DNP\nR_{3} = 10 kΩ\n"
+    (at 228.6 102.87 0)
+    (effects (font (size 1.27 1.27)) (justify left bottom))
+  )
   (text "See:\n9.2.1.2.1 Series and Parallel Resonant Capacitor Selection"
     (at 29.21 73.66 0)
@@
     )
   )
+  (global_label "Qi_TS{slash}CTRL" (shape input) (at 193.04 148.59 0) (fields_autoplaced)
+    (effects (font (size 1.27 1.27)) (justify left))
+    (property "Intersheet References" "${INTERSHEET_REFS}" (id 0) (at 206.3104 148.5106 0)
+      (effects (font (size 1.27 1.27)) (justify left) hide)
+    )
+  )
   (global_label "~{Qi_CHG{slash}LED}" (shape bidirectional) (at 233.68 40.64 0) (fields_autoplaced)
     (effects (font (size 1.27 1.27)) (justify left))
@@
     )
   )
+  (global_label "Qi_TS{slash}CTRL" (shape output) (at 231.14 64.77 0) (fields_autoplaced)
+    (effects (font (size 1.27 1.27)) (justify left))
+    (property "Intersheet References" "${INTERSHEET_REFS}" (id 0) (at 244.4104 64.6906 0)
+      (effects (font (size 1.27 1.27)) (justify left) hide)
+    )
+  )
   (global_label "LED_V+" (shape input) (at 54.61 137.16 180) (fields_autoplaced)
     (effects (font (size 1.27 1.27)) (justify right))
@@
   (symbol (lib_id "Device:R_Small") (at 220.98 59.69 0) (unit 1)
     (in_bom yes) (on_board yes) (fields_autoplaced)
-    (property "Reference" "R2" (id 0) (at 223.52 58.4199 0)
+    (property "Reference" "R2" (id 0) (at 223.52 55.8799 0)
       (effects (font (size 1.27 1.27)) (justify left))
     )
-    (property "Value" "20k" (id 1) (at 223.52 60.9599 0)
+    (property "Value" "20k" (id 1) (at 223.52 58.4199 0)
       (effects (font (size 1.27 1.27)) (justify left))
     )
@@
       (effects (font (size 1.27 1.27)) hide)
     )
-    (property "Name" "" (id 4) (at 223.52 62.2299 0)
-      (effects (font (size 1.27 1.27)) (justify left) hide)
+    (property "fit_field" "DNP" (id 4) (at 223.52 60.9599 0)
+      (effects (font (size 1.27 1.27)) (justify left))
+    )
+    (property "Name" "R_{2NTC}" (id 5) (at 223.52 63.4999 0)
+      (effects (font (size 1.27 1.27)) (justify left))
     )
     (pin "1")
@@
   (symbol (lib_id "Device:R_Small") (at 220.98 69.85 0) (unit 1)
     (in_bom yes) (on_board yes) (fields_autoplaced)
-    (property "Reference" "R3" (id 0) (at 223.52 68.5799 0)
+    (property "Reference" "R3" (id 0) (at 223.52 66.0399 0)
       (effects (font (size 1.27 1.27)) (justify left))
     )
-    (property "Value" "R" (id 1) (at 223.52 71.1199 0)
+    (property "Value" "464k" (id 1) (at 223.52 68.5799 0)
       (effects (font (size 1.27 1.27)) (justify left))
     )
@@
       (effects (font (size 1.27 1.27)) hide)
     )
-    (property "Name" "" (id 4) (at 223.52 72.3899 0)
-      (effects (font (size 1.27 1.27)) (justify left) hide)
+    (property "fit_field" "DNP" (id 4) (at 223.52 71.1199 0)
+      (effects (font (size 1.27 1.27)) (justify left))
+    )
+    (property "Name" "R_{1NTC}" (id 4) (at 223.52 73.6599 0)
+      (effects (font (size 1.27 1.27)) (justify left))
     )
     (pin "1")
@@
     (pin "1")
   )
-  (symbol (lib_id "power:GND") (at 177.8 60.96 0) (unit 1)
-    (in_bom yes) (on_board yes) (fields_autoplaced)
-    (property "Reference" "#PWR011" (id 0) (at 177.8 67.31 0)
-      (effects (font (size 1.27 1.27)) hide)
-    )
-    (property "Value" "GND" (id 1) (at 177.8 66.04 0))
-    (property "Footprint" "" (id 2) (at 177.8 60.96 0)
-      (effects (font (size 1.27 1.27)) hide)
-    )
-    (property "Datasheet" "" (id 3) (at 177.8 60.96 0)
-      (effects (font (size 1.27 1.27)) hide)
-    )
-    (pin "1")
-  )
   (symbol (lib_id "Device:C_Small") (at 175.26 29.21 0) (unit 1)
     (in_bom yes) (on_board yes) (fields_autoplaced)
@@
     (pin "2")
   )
-  (symbol (lib_id "Connector_Generic:Conn_01x02") (at 238.76 74.93 0) (unit 1)
+  (symbol (lib_id "Connector_Generic:Conn_01x02") (at 238.76 77.47 0) (mirror x) (unit 1)
     (in_bom yes) (on_board yes) (fields_autoplaced)
     (property "Reference" "J3" (id 0) (at 241.3 74.9299 0)
       (effects (font (size 1.27 1.27)) (justify left))
     )
-    (property "Value" "Conn_01x02" (id 1) (at 241.3 76.1999 0)
+    (property "Value" "Conn_01x02" (id 1) (at 241.3 76.2001 0)
       (effects (font (size 1.27 1.27)) (justify left) hide)
     )
-    (property "Footprint" "Connector_PinHeader_2.54mm:PinHeader_1x02_P2.54mm_Vertical" (id 2) (at 238.76 74.93 0)
+    (property "Footprint" "Connector_PinHeader_2.54mm:PinHeader_1x02_P2.54mm_Vertical" (id 2) (at 238.76 77.47 0)
       (effects (font (size 1.27 1.27)) hide)
     )
-    (property "Datasheet" "~" (id 3) (at 238.76 74.93 0)
+    (property "Datasheet" "~" (id 3) (at 238.76 77.47 0)
       (effects (font (size 1.27 1.27)) hide)
     )
@@
       (effects (font (size 1.27 1.27)) (justify left))
     )
-    (property "fit_field" "DNP" (id 5) (at 238.76 74.93 0)
+    (property "fit_field" "DNP" (id 5) (at 238.76 77.47 0)
       (effects (font (size 1.27 1.27)) hide)
     )
@@
       (effects (font (size 1.27 1.27)) hide)
     )
-    (property "Name" "C_{3}" (id 4) (at 205.74 76.2062 0)
+    (property "Name" "C_{3NTC}" (id 4) (at 205.74 76.2062 0)
       (effects (font (size 1.27 1.27)) (justify left))
     )
@@
   (symbol (lib_id "Device:R_Small") (at 212.09 73.66 0) (unit 1)
     (in_bom yes) (on_board yes) (fields_autoplaced)
-    (property "Reference" "R6" (id 0) (at 214.63 72.3899 0)
+    (property "Reference" "R6" (id 0) (at 214.63 71.1199 0)
       (effects (font (size 1.27 1.27)) (justify left))
     )
-    (property "Value" "R" (id 1) (at 214.63 74.9299 0)
+    (property "Value" "10k" (id 1) (at 214.63 73.6599 0)
       (effects (font (size 1.27 1.27)) (justify left))
     )
@@
       (effects (font (size 1.27 1.27)) hide)
     )
-    (property "Name" "" (id 4) (at 214.63 76.1999 0)
-      (effects (font (size 1.27 1.27)) (justify left) hide)
+    (property "Name" "R_{3NTC}" (id 4) (at 214.63 76.1999 0)
+      (effects (font (size 1.27 1.27)) (justify left))
     )
     (pin "1")
@@
       (reference "#PWR010") (unit 1) (value "+BATT") (footprint "")
     )
-    (path "/b114816e-d3b3-4d0f-ac43-e555d80a8a01"
-      (reference "#PWR011") (unit 1) (value "GND") (footprint "")
-    )
     (path "/4fc81e6c-b0af-46d4-9130-636f21c7500a"
       (reference "#PWR012") (unit 1) (value "GND") (footprint "")
@@
     )
     (path "/ad9bdf3d-d3b2-4f66-860f-7d019cc33f16"
-      (reference "R3") (unit 1) (value "R") (footprint "Resistor_SMD:R_0603_1608Metric")
+      (reference "R3") (unit 1) (value "464k") (footprint "Resistor_SMD:R_0603_1608Metric")
     )
     (path "/fb0a85bb-e074-43a2-8ad1-7e5f7e93e678"
@@
     )
     (path "/ec1d3a47-69bb-4c48-bede-986703428dd5"
-      (reference "R6") (unit 1) (value "R") (footprint "Resistor_SMD:R_0603_1608Metric")
+      (reference "R6") (unit 1) (value "10k") (footprint "Resistor_SMD:R_0603_1608Metric")
     )
     (path "/325888c5-0937-48d4-8189-9d8dbc457f48"

Commit message: Moving in
Parts:
- JP1: renamed from JP5; fit_field (none) -> DNP
- JP10: renamed from JP14; fit_field (none) -> DNP
- JP11: renamed from JP4; fit_field (none) -> DNP
- JP12: renamed from JP1; fit_field (none) -> DNP
- JP2: renamed from JP6; fit_field (none) -> DNP
- JP3: renamed from JP7; fit_field (none) -> DNP
- JP4: renamed from JP8; fit_field (none) -> DNP
- JP5: renamed from JP9; fit_field (none) -> DNP
- JP6: renamed from JP10; fit_field (none) -> DNP
- JP7: renamed from JP11; fit_field (none) -> DNP
- JP8: renamed from JP12; fit_field (none) -> DNP
- JP9: renamed from JP13; fit_field (none) -> DNP

Commit message: Puzzling
Parts:
- removed J1, J3: Conn_01x02, Connector_PinHeader_2.54mm:PinHeader_1x02_P2.54mm_Vertical, symbol Connector_Generic:Conn_01x02
- added J1: Conn_01x03, Connector_PinHeader_2.54mm:PinHeader_1x03_P2.54mm_Vertical, symbol Connector_Generic:Conn_01x03
Connections:
- net +BATT: now also J1.1 (Pin_1)
- net GND: now also C27.1, J1.3 (Pin_3); no longer C27.2
- net LED_V+: now also C27.2; no longer C27.1
- net ~{Qi_CHG/LED}: now also U3.11 (GPIO9); no longer U3.20 (GPIO5)
- net Qi_NTC renamed NTC
- net NTC: now also J1.2 (Pin_2)
Other:
- moved on the sheet: D11, R2, R3, R4

Commit message: Puzzling #2
Parts:
- J1: Name (none) -> Battery
- TP1: footprint Connector_PinHeader_2.54mm:PinHeader_1x02_P2.54mm_Vertical -> Connector_PinHeader_1.00mm:PinHeader_1x02_P1.00mm_Vertical
Connections:
- net +BATT: now also J1.3 (Pin_3); no longer J1.1 (Pin_1)
- net GND: now also J1.1 (Pin_1); no longer J1.3 (Pin_3)
Changed lines of the file:
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@@
     (comment 3 "Danmark")
     (comment 4 "www.step7.dk")
-    (comment 5 "Qi Lamp Board")
+    (comment 5 "Qi WiFi Lamp")
     (comment 6 "ESP8266_Lampe")
     (comment 7 "Martin")
@@
     (pin "1")
   )
-  (symbol (lib_id "Connector_Generic:Conn_01x03") (at 64.77 167.64 0) (unit 1)
-    (in_bom yes) (on_board yes)
-    (property "Reference" "J1" (id 0) (at 67.31 166.3699 0)
-      (effects (font (size 1.27 1.27)) (justify left))
-    )
-    (property "Value" "Conn_01x03" (id 1) (at 67.31 167.6399 0)
+  (symbol (lib_id "Connector_Generic:Conn_01x03") (at 64.77 167.64 0) (mirror x) (unit 1)
+    (in_bom yes) (on_board yes) (fields_autoplaced)
+    (property "Reference" "J1" (id 0) (at 64.77 158.75 0))
+    (property "Value" "Conn_01x03" (id 1) (at 67.31 167.6401 0)
       (effects (font (size 1.27 1.27)) (justify left) hide)
     )
@@
       (effects (font (size 1.27 1.27)) hide)
     )
-    (property "silk_text" "B+ _{NTC} B-" (id 4) (at 67.31 168.9099 0)
-      (effects (font (size 1.27 1.27)) (justify left))
+    (property "silk_text" "B+ _{NTC} B-" (id 4) (at 67.31 166.3701 0)
+      (effects (font (size 1.27 1.27)) (justify left) hide)
     )
     (property "fit_field" "DNP" (id 5) (at 64.77 167.64 0)
       (effects (font (size 1.27 1.27)) hide)
     )
+    (property "Name" "Battery" (id 6) (at 64.77 161.29 0))
     (pin "1")
     (pin "2")
@@
       (effects (font (size 1.27 1.27)) (justify left) hide)
     )
-    (property "Footprint" "Connector_PinHeader_2.54mm:PinHeader_1x02_P2.54mm_Vertical" (id 2) (at 252.73 123.19 0)
+    (property "Footprint" "Connector_PinHeader_1.00mm:PinHeader_1x02_P1.00mm_Vertical" (id 2) (at 252.73 123.19 0)
       (effects (font (size 1.27 1.27)) hide)
     )
@@
     )
     (path "/da7e2678-b00f-46fb-93d1-64bc4ee7cebe"
-      (reference "TP1") (unit 1) (value "TestPoint_2Pole") (footprint "Connector_PinHeader_2.54mm:PinHeader_1x02_P2.54mm_Vertical")
+      (reference "TP1") (unit 1) (value "TestPoint_2Pole") (footprint "Connector_PinHeader_1.00mm:PinHeader_1x02_P1.00mm_Vertical")
     )
     (path "/30c5f696-f195-43bd-8ac9-7362f9499192"

Commit message: Puzzling #3
Parts:
- TP1: footprint Connector_PinHeader_1.00mm:PinHeader_1x02_P1.00mm_Vertical -> Connector_PinHeader_1.27mm:PinHeader_1x02_P1.27mm_Vertical
Connections:
- net GND: now also C26.1, C30.2; no longer C26.2, C30.1
- net LED_V+: now also C26.2, C30.1; no longer C26.1, C30.2
Changed lines of the file:
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@@
     (pin "9")
   )
-  (symbol (lib_id "Device:C_Small") (at 255.27 208.28 0) (mirror x) (unit 1)
-    (in_bom yes) (on_board yes) (fields_autoplaced)
-    (property "Reference" "C30" (id 0) (at 252.73 207.0035 0)
-      (effects (font (size 1.27 1.27)) (justify right))
-    )
-    (property "Value" "330n" (id 1) (at 252.73 209.5435 0)
-      (effects (font (size 1.27 1.27)) (justify right))
+  (symbol (lib_id "Device:C_Small") (at 255.27 208.28 0) (mirror y) (unit 1)
+    (in_bom yes) (on_board yes) (fields_autoplaced)
+    (property "Reference" "C30" (id 0) (at 252.73 207.0162 0)
+      (effects (font (size 1.27 1.27)) (justify left))
+    )
+    (property "Value" "330n" (id 1) (at 252.73 209.5562 0)
+      (effects (font (size 1.27 1.27)) (justify left))
     )
     (property "Footprint" "Capacitor_SMD:C_0603_1608Metric" (id 2) (at 255.27 208.28 0)
@@
     (pin "2")
   )
-  (symbol (lib_id "Device:C_Small") (at 113.03 208.28 0) (mirror y) (unit 1)
-    (in_bom yes) (on_board yes) (fields_autoplaced)
-    (property "Reference" "C26" (id 0) (at 110.49 207.0162 0)
-      (effects (font (size 1.27 1.27)) (justify left))
-    )
-    (property "Value" "330n" (id 1) (at 110.49 209.5562 0)
-      (effects (font (size 1.27 1.27)) (justify left))
+  (symbol (lib_id "Device:C_Small") (at 113.03 208.28 0) (mirror x) (unit 1)
+    (in_bom yes) (on_board yes) (fields_autoplaced)
+    (property "Reference" "C26" (id 0) (at 110.49 207.0035 0)
+      (effects (font (size 1.27 1.27)) (justify right))
+    )
+    (property "Value" "330n" (id 1) (at 110.49 209.5435 0)
+      (effects (font (size 1.27 1.27)) (justify right))
     )
     (property "Footprint" "Capacitor_SMD:C_0603_1608Metric" (id 2) (at 113.03 208.28 0)
@@
       (effects (font (size 1.27 1.27)) (justify left) hide)
     )
-    (property "Footprint" "Connector_PinHeader_1.00mm:PinHeader_1x02_P1.00mm_Vertical" (id 2) (at 252.73 123.19 0)
+    (property "Footprint" "Connector_PinHeader_1.27mm:PinHeader_1x02_P1.27mm_Vertical" (id 2) (at 252.73 123.19 0)
       (effects (font (size 1.27 1.27)) hide)
     )
@@
     )
     (path "/da7e2678-b00f-46fb-93d1-64bc4ee7cebe"
-      (reference "TP1") (unit 1) (value "TestPoint_2Pole") (footprint "Connector_PinHeader_1.00mm:PinHeader_1x02_P1.00mm_Vertical")
+      (reference "TP1") (unit 1) (value "TestPoint_2Pole") (footprint "Connector_PinHeader_1.27mm:PinHeader_1x02_P1.27mm_Vertical")
     )
     (path "/30c5f696-f195-43bd-8ac9-7362f9499192"

Commit message: Puzzling #4
Other:
- note added: "When DTR is released C_{on} = 100n takes around 1 second to fall below V_{ON} < 0.3 V through internal 4 MΩ pull down resistor of SLG5NV1430V"
- note removed: "C_{on} = 100n gives around 1 second to fall below V_{ON} < 0.3 V through internal 4 MΩ pull down resistor of SLG5NV1430V"
Changed lines of the file:
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@@
     (effects (font (size 1.27 1.27)) (justify left bottom))
   )
-  (text "C_{on} = 100n gives around 1 second to fall below V_{ON} < 0.3 V through internal 4 MΩ pull down resistor of SLG5NV1430V"
+  (text "When DTR is released C_{on} = 100n takes around 1 second to fall below V_{ON} < 0.3 V\nthrough internal 4 MΩ pull down resistor of SLG5NV1430V"
     (at 261.62 74.93 0)
     (effects (font (size 1.27 1.27)) (justify left bottom))
