File: qi-lamp-charger.kicad_sch (KiCad schematic)
At the start: 84 parts, among them J1 Conn_01x03, J2 Conn_01x02, J4 Conn_01x06, J5 Conn_01x03, Q1 BSS308PE H6327, SW1 SKTDLDE010, U1 SLG5NV1430V, U2 BQ51050BRHL, U3 ESP-12E

Commit message: Shematic changed
Parts:
- removed JP12: SolderJumper_2_Bridged, Jumper:SolderJumper-2_P1.3mm_Bridged_RoundedPad1.0x1.5mm, symbol Jumper:SolderJumper_2_Bridged
- added D? (x2): CD0603-B0340R, Diode_SMD:D_0603_1608Metric, symbol Device:D_Small_Filled
- added R15, R?: 20k, Resistor_SMD:R_0603_1608Metric, symbol Device:R_Small
- added R?: 340k, Resistor_SMD:R_0603_1608Metric, symbol Device:R_Small
- added R?: 100k, Resistor_SMD:R_0603_1608Metric, symbol Device:R_Small
- TP1: fit_field DNP -> man_rst; silk_text man_rst -> Bootloader
Connections:
- net ESP_GPIO0 is gone; now on net DTR: R11.1, U3.18 (GPIO0)
- net +VSW: now also R?.2, R?.2
- net DTR: now also TP1.2
- net GND: now also R?.1
- net NTC: no longer U3.2 (ADC)
- net Qi_TS/CTRL: now also U3.20 (GPIO5); no longer U3.7 (GPIO13)
- net RTS: now also U3.1 (~{RST})
- net ~{Qi_CHG/LED}: now also D?.1 (K), R15.1; no longer R4.1, U2.7 (~{CHG})
- net BTN: no longer names the net of Q1.1 (G), R14.1
- net BTN: now also D?.2 (A), D?.2 (A); no longer SW1.2, U3.5 (GPIO14)
- net PWR_ON/~{OFF} renamed KEEP_ALIVE
- removed net ~{ESP_RST}: TP1.2, U3.1 (~{RST})
- new net: R15.2, R4.1, U2.7 (~{CHG})
- new net BAT_ADC: R?.1, R?.2, U3.2 (ADC)
- new net ~{BTN}: D?.1 (K), R?.1, SW1.2, U3.5 (GPIO14)
Other:
- note added: "ADC0 (Read) Read battery voltage, range: 4.40V GPIO1 (Write) UART GPIO2 (Write) LED string data out GPIO3 (Read) UART GPIO4 (Write) Power switch control: high=run, low=stop, released=stop w. delay GPIO9 (Read) Qi charging status: high=off, low=on GPIO9 (Write) Qi status LED D11: high=off, low=on GPIO12 (Read) LED string data return (optional, for errorchecking) GPIO13 (Read) Qi NTC status - if pr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"
- note added: "Design values for NTC: β = 3534 R_{o} = 10 kΩ R_{1} = 200 Ω R_{2} = 20 kΩ R_{3} = 464 kΩ Without NTC: R_{2} = DNP R_{3} = 10 kΩ Reference: bq5105xB datasheet and TS_ Calculator Tool Rev A"
- note added: "Flashing auto_rst mode requires RST and DTR man_rst mode does not use RST and DTR Reference: https://circuitjournal.com/esp8266-with-arduino-ide#connecting-via-usb"
- note added: "RTS RXD TXD n/c DTR GND"
- note added: "When Q1 is released then C_{on} = 100n will take around 1 second to fall below V_{ON} > 0.3 V C_{on} is discharged through internal 4 MΩ pull down resistor of SLG5NV1430V"
- note removed: "Design for NTC: NTC β = 3534 NTC Ro = 10 kΩ R_{1} = 200 Ω R_{2} = 20 kΩ R_{3} = 464 kΩ No NTC: R_{2} = DNP R_{3} = 10 kΩ"
- note removed: "GND DTR n/c TXD RXD RTS"
- note removed: "Programming reference: https://circuitjournal.com/esp8266-with-arduino-ide#connecting-via-usb"
- note removed: "When DTR is released C_{on} = 100n takes around 1 second to fall below V_{ON} < 0.3 V through internal 4 MΩ pull down resistor of SLG5NV1430V"
- moved on the sheet: C12, C16, C22, C34, C8, J4, Q1, R10, R12, R14, R9, SW1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

Commit message: Puzzle #6
Parts:
- removed H1, H2, H3: MountingHole, MountingHole:MountingHole_3.2mm_M3_ISO14580, symbol Mechanical:MountingHole
- gave numbers to parts that had none: 5
Other:
- note added: "Pin definitions: ADC0 (Read) Read battery voltage, range: 4.40V GPIO1 (Write) UART GPIO2 (Write) LED string data out GPIO3 (Read) UART GPIO4 (Write) Power switch control: high=run, low=stop, released=stop w. delay GPIO9 (Read) Qi charging status: high=off, low=on GPIO9 (Write) Qi status LED D11: high=off, low=on GPIO12 (Read) LED string data return (optional, for errorchecking) GPIO13 (Read) Qi N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"
- note added: "Reference: https://randomnerdtutorials.com/esp8266-pinout-reference-gpios/"
- note removed: "ADC0 (Read) Read battery voltage, range: 4.40V GPIO1 (Write) UART GPIO2 (Write) LED string data out GPIO3 (Read) UART GPIO4 (Write) Power switch control: high=run, low=stop, released=stop w. delay GPIO9 (Read) Qi charging status: high=off, low=on GPIO9 (Write) Qi status LED D11: high=off, low=on GPIO12 (Read) LED string data return (optional, for errorchecking) GPIO13 (Read) Qi NTC status - if pr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"
- moved on the sheet: C23, J1, J4, J5, R17, R18

Commit message: Add info
Parts:
- C1: Manufacturer_Name (none) -> Samsung; Name (none) -> C_{s3}
- C10: Manufacturer_Name (none) -> Samsung; Manufacturer_Part_Number (none) -> CL10B473KO8NNND; Name (none) -> C_{comm1}; silk_text C_{comm1} -> (none)
- C11: Manufacturer_Name (none) -> Samsung; Manufacturer_Part_Number (none) -> CL10B103KO8NNNC; Name (none) -> C_{boot1}; silk_text C_{boot1} -> (none)
- C12, C13, C3, C34, C4, C8: Manufacturer_Name (none) -> Samsung; Manufacturer_Part_Number (none) -> CL10B104KO8NNND
- C14: Manufacturer_Name (none) -> Samsung; Name (none) -> C_{p2}; Rating (none) -> 50V
- C15: Manufacturer_Name (none) -> Samsung; Name (none) -> C_{p3}; Rating (none) -> 50V
- C16: Manufacturer_Name (none) -> Samsung; Manufacturer_Part_Number (none) -> CL10B104KO8NNND; Name (none) -> C_{on}; silk_text C_{on} -> (none)
- C17: Manufacturer_Name (none) -> Samsung; Manufacturer_Part_Number (none) -> CL10B103KO8NNNC; Name (none) -> C_{boot2}; silk_text C_{boot2} -> (none)
- C18: Manufacturer_Name (none) -> Samsung; Manufacturer_Part_Number (none) -> CL10B473KO8NNND; Name (none) -> C_{comm2}; silk_text C_{comm2} -> (none)
- C19: Manufacturer_Name (none) -> Samsung; Manufacturer_Part_Number (none) -> CL10B474KO8NNNC; Name (none) -> C_{clamp2}; silk_text C_{clamp2} -> (none)
- C2: Manufacturer_Name (none) -> Samsung; Name (none) -> C_{p1}; Rating (none) -> 50V
- C20, C21, C22: Manufacturer_Name (none) -> Samsung; Manufacturer_Part_Number (none) -> CL21A106KOQNNNE
- C23, C24, C25, C26, C27, C28, C29, C30, C31, C32, C33: Manufacturer_Name (none) -> Samsung; Manufacturer_Part_Number (none) -> CL10B334KO8NNNC
- C5: Manufacturer_Name (none) -> Samsung; Manufacturer_Part_Number (none) -> CL10A105KO8NNNC
- C6: Manufacturer_Name (none) -> Samsung; Name (none) -> C_{s1}
- C7: Manufacturer_Name (none) -> Samsung; Name (none) -> C_{s2}
- C9: Manufacturer_Name (none) -> Samsung; Manufacturer_Part_Number (none) -> CL10B474KO8NNNC; Name (none) -> C_{clamp1}; silk_text C_{clamp1} -> (none)
- D1, D10, D2, D3, D4, D5, D6, D7, D8, D9: Manufacturer_Name (none) -> DONGGUAN OCCIDENTAL; Manufacturer_Part_Number (none) -> SK6812
- D11: value LED_Green -> LED_Red; Manufacturer_Name (none) -> Lite-On; Manufacturer_Part_Number (none) -> LTST-C191KFKT
- D12, D13: Manufacturer_Name (none) -> Bourns; Manufacturer_Part_Number (none) -> CD0603-B0340R
- J1: silk_text B+ _{NTC} B- -> (none)
- J2: Name (none) -> RxCoil; silk_text RxCoil -> (none)
- J4: Name (none) -> Serial; silk_text Serial -> (none)
- J5: Name (none) -> External strip; silk_text External strip -> (none)
- JP11: Name (none) -> LED-V_{bat}; silk_text LED-V_{bat} -> (none)
- Q1: Manufacturer_Name (none) -> Infineon; Manufacturer_Part_Number (none) -> BSS308PE H6327
- R1: Manufacturer_Name (none) -> Panasonic; Manufacturer_Part_Number (none) -> ERJ-3EKF2050V; Name (none) -> R_{ilim}; silk_text R_{ilim} -> (none)
- R10, R11: Manufacturer_Name (none) -> Panasonic; Manufacturer_Part_Number (none) -> ERJ-3EKF2002V; Name (none) -> auto_rst
- R12, R13, R14, R15, R16, R2, R9: Manufacturer_Name (none) -> Panasonic; Manufacturer_Part_Number (none) -> ERJ-3EKF2002V
- R17: Manufacturer_Name (none) -> Panasonic; Manufacturer_Part_Number (none) -> ERJ-3EKF3403V
- R18: Manufacturer_Name (none) -> Panasonic; Manufacturer_Part_Number (none) -> ERJ-3EKF1003V
- R3: Manufacturer_Name (none) -> Panasonic; Manufacturer_Part_Number (none) -> ERJ-3EKF4643V
- R4: Manufacturer_Name (none) -> Panasonic; Manufacturer_Part_Number (none) -> ERJ-3EKF1000V
- R5: Manufacturer_Name (none) -> Panasonic; Manufacturer_Part_Number (none) -> ERJ-3EKF2401V; Name (none) -> R_{term}; silk_text R_{term} -> (none)
- R6: Manufacturer_Name (none) -> Panasonic; Manufacturer_Part_Number (none) -> ERJ-3EKF1002V
- R7: Manufacturer_Name (none) -> Panasonic; Manufacturer_Part_Number (none) -> ERJ-3EKF2002V; Name (none) -> R_{os}; silk_text R_{os} -> (none)
- R8: Manufacturer_Name (none) -> Panasonic; Manufacturer_Part_Number (none) -> ERJ-3EKF2000V; Name (none) -> R_{fod}; silk_text R_{fod} -> (none)
- SW1: Manufacturer_Name (none) -> ALPS; Manufacturer_Part_Number (none) -> SKTDLDE010
- TP1: Name (none) -> Bootloader; silk_text Bootloader -> (none)
- U1: Manufacturer_Name (none) -> Renesas; Manufacturer_Part_Number (none) -> SLG5NV1430V
- U2: Manufacturer_Name (none) -> Texas Instruments; Manufacturer_Part_Number (none) -> BQ51050BRHLR
Other:
- note added: "TDK WR464650-10K2-FS3 46x46x2.97 7.3uH / 0.07R 7,66 € TDK WR444030-16F3-G 40x44x0.62 19uH / 0.70R 5,93 € TDK WR424245-13K2-G 42x42x0.91 11.9uH / 0.22R 6,77 € TDK WR303050-12F5-ID 30.4x30x0.92 12.3uH / 0.41R 4,62 € TDK WR303050-12F5-ID 30.4x30x0.94 8.23uH / 0.28R 4,96 € Pulse WMRR138F-0 (YZ-ZR3832) 32x38x0.27 12.5uH / 0.32R 2,95 € Pulse WMRR132F-0 Ø30x0.22 11.5uH / 0.59R 3,56 €"
- moved on the sheet: C1, C14, C15, C2, C6, C7, J2

Commit message: As ordered
Parts:
- added H1, H2: MountingHole, MountingHole:MountingHole_2.2mm_M2, symbol Mechanical:MountingHole
- Q1: value BSS308PE H6327 -> BSS 209PW; Manufacturer_Part_Number BSS308PE H6327 -> BSS209PWH6327XTSA1
Changed lines of the file:
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@@
     (pin "2")
+  )
+  (symbol (lib_id "Mechanical:MountingHole") (at 52.07 274.32 0) (unit 1)
+    (in_bom yes) (on_board yes) (fields_autoplaced)
+    (property "Reference" "H2" (id 0) (at 54.61 273.0499 0)
+      (effects (font (size 1.27 1.27)) (justify left))
+    )
+    (property "Value" "MountingHole" (id 1) (at 54.61 275.5899 0)
+      (effects (font (size 1.27 1.27)) (justify left))
+    )
+    (property "Footprint" "MountingHole:MountingHole_2.2mm_M2" (id 2) (at 52.07 274.32 0)
+      (effects (font (size 1.27 1.27)) hide)
+    )
+    (property "Datasheet" "~" (id 3) (at 52.07 274.32 0)
+      (effects (font (size 1.27 1.27)) hide)
+    )
   )
   (symbol (lib_id "power:GND") (at 290.83 212.09 0) (mirror y) (unit 1)
@@
     (pin "2")
   )
+  (symbol (lib_id "Mechanical:MountingHole") (at 26.67 274.32 0) (unit 1)
+    (in_bom yes) (on_board yes) (fields_autoplaced)
+    (property "Reference" "H1" (id 0) (at 29.21 273.0499 0)
+      (effects (font (size 1.27 1.27)) (justify left))
+    )
+    (property "Value" "MountingHole" (id 1) (at 29.21 275.5899 0)
+      (effects (font (size 1.27 1.27)) (justify left))
+    )
+    (property "Footprint" "MountingHole:MountingHole_2.2mm_M2" (id 2) (at 26.67 274.32 0)
+      (effects (font (size 1.27 1.27)) hide)
+    )
+    (property "Datasheet" "~" (id 3) (at 26.67 274.32 0)
+      (effects (font (size 1.27 1.27)) hide)
+    )
+  )
   (symbol (lib_id "power:GND") (at 193.04 81.28 0) (unit 1)
     (in_bom yes) (on_board yes) (fields_autoplaced)
@@
       (effects (font (size 1.27 1.27)) (justify left))
     )
-    (property "Value" "BSS308PE H6327" (id 1) (at 307.34 40.6399 0)
+    (property "Value" "BSS 209PW" (id 1) (at 307.34 40.6399 0)
       (effects (font (size 1.27 1.27)) (justify left))
     )
@@
       (effects (font (size 1.27 1.27)) hide)
     )
-    (property "Manufacturer_Part_Number" "BSS308PE H6327" (id 6) (at 300.99 40.64 0)
+    (property "Manufacturer_Part_Number" "BSS209PWH6327XTSA1" (id 6) (at 300.99 40.64 0)
       (effects (font (size 1.27 1.27)) hide)
     )
@@
       (reference "D13") (unit 1) (value "CD0603-B0340R") (footprint "Diode_SMD:D_0603_1608Metric")
     )
+    (path "/5b25914f-da9d-4cc2-a32e-623eaa28c78a"
+      (reference "H1") (unit 1) (value "MountingHole") (footprint "MountingHole:MountingHole_2.2mm_M2")
+    )
+    (path "/2f6e5e60-a129-477c-a20a-b88ba73ca44b"
+      (reference "H2") (unit 1) (value "MountingHole") (footprint "MountingHole:MountingHole_2.2mm_M2")
+    )
     (path "/5692bf59-80e3-4420-a260-8a77be664c2a"
       (reference "J1") (unit 1) (value "Conn_01x03") (footprint "Connector_PinHeader_2.54mm:PinHeader_1x03_P2.54mm_Vertical")
@@
     )
     (path "/8d372b16-e071-48c6-a79d-fb34910a7f02"
-      (reference "Q1") (unit 1) (value "BSS308PE H6327") (footprint "Package_TO_SOT_SMD:SOT-23")
+      (reference "Q1") (unit 1) (value "BSS 209PW") (footprint "Package_TO_SOT_SMD:SOT-23")
     )
     (path "/9d075e4e-fa2a-4634-8e55-c819d887aebb"
